File: CADfiles/MasterOfMuppets/unripple_module.kicad_sch (KiCad schematic)
At the start: 2 parts

Commit message: PCB Preps
Re-assigned footprints;
Placed all symbols in the middle;
Removed instruction to ignore the PCB in the README.manahmanah;
Added a generic placement recommendation file from Sir. Claude;
Ready to start the design;
Parts:
- C21: footprint 4ms_Capacitor:C_0603 -> PCM_4ms_Capacitor:C_0603
- C22: footprint 4ms_Capacitor:C_0805 -> PCM_4ms_Capacitor:C_0805
Changed lines of the file:
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@@
 			)
 		)
-		(property "Footprint" "4ms_Capacitor:C_0805"
+		(property "Footprint" "PCM_4ms_Capacitor:C_0805"
 			(at 101.6 72.39 0)
 			(effects
@@
 			)
 		)
-		(property "Footprint" "4ms_Capacitor:C_0603"
+		(property "Footprint" "PCM_4ms_Capacitor:C_0603"
 			(at 87.63 72.39 0)
 			(effects
