File: CADfiles/MasterOfMuppets/MasterOfMuppets.kicad_pcb (KiCad board)
At the start: 2 copper layers, 71.1 x 111.8 mm, 73 parts, among them T1 Teensy4.1

Commit message: Let there be light
said the voice in the void
Parts:
- removed C1, C2, C3, C5: 0.1uf, Capacitor_THT:C_Disc_D5.0mm_W2.5mm_P5.00mm
- removed C4: 1uf, Capacitor_THT:C_Disc_D5.0mm_W2.5mm_P5.00mm
- removed DAC1, DAC2, DAC3: MCP4728, Package_SO:MSOP-10_3x3mm_P0.5mm
- removed Eurorack1: ~, Connector_IDC:IDC-Header_2x08_P2.54mm_Vertical
- removed G***: LOGO, LOGO
- removed OUT_CV1, OUT_CV10, OUT_CV11, OUT_CV12, OUT_CV2, OUT_CV3, OUT_CV4, OUT_CV5, OUT_CV6, OUT_CV7, OUT_CV8, OUT_CV9: ACJM-MV35-2S, PCM_4ms_Jack:ACJM-MV35-2S_Mono_Vert_Switch
- removed OpAmp1, OpAmp2, OpAmp3: TL074, Package_DIP:DIP-14_W7.62mm_Socket
- removed R1, R11, R12, R2, R22, R23, R24, R25, R42, R43, R44, R45: 1k, Resistor_THT:R_Axial_DIN0204_L3.6mm_D1.6mm_P1.90mm_Vertical
- removed R10, R26, R27, R28, R29, R3, R30, R31, R32, R33, R34, R35, R36, R37, R38, R39, R4, R40, R41, R5, R6, R7, R8, R9: 47k, Resistor_THT:R_Axial_DIN0204_L3.6mm_D1.6mm_P1.90mm_Vertical
- removed R13, R15, R17, R19, R20, R21: 10k, Resistor_THT:R_Axial_DIN0204_L3.6mm_D1.6mm_P1.90mm_Vertical
- removed R14, R16, R18: 100k, Resistor_THT:R_Axial_DIN0204_L3.6mm_D1.6mm_P1.90mm_Vertical
- removed T1: Teensy4.1, teensy.pretty-master:Teensy41
- removed USB Through: , Connector_PinHeader_2.54mm:PinHeader_2x04_P2.54mm_Vertical
- removed V_REG1: LD1117V50, PCM_4ms_Package_TO:TO-220-3_Vertical
Routing:
- net GND: track 639.5 -> 0.00 mm
- net VCC: track 234.7 -> 0.00 mm, vias 4 -> 0
- net +12V: track 186.7 -> 0.00 mm, vias 2 -> 0
- net /BOODOO_BOARD2/CV_1: track 117.5 -> 0.00 mm
- net /BOODOO_BOARD/RDY_~{BSY}: track 101.2 -> 0.00 mm
- net /BOODOO_BOARD/~{LDAC}: track 99.5 -> 0.00 mm
- net /BOODOO_BOARD/SDA: track 95.0 -> 0.00 mm
- net /BOODOO_BOARD/SCL: track 84.9 -> 0.00 mm
- net /BOODOO_BOARD/CV_3: track 82.5 -> 0.00 mm, vias 1 -> 0
- net /BOODOO_BOARD2/~{LDAC}: track 69.0 -> 0.00 mm
- net /BOODOO_BOARD1/CV_2: track 68.1 -> 0.00 mm
- net /BOODOO_BOARD2/RDY_~{BSY}: track 59.0 -> 0.00 mm
- net /BOODOO_BOARD1/SCL: track 59.0 -> 0.00 mm
- net /BOODOO_BOARD/CV_4: track 57.6 -> 0.00 mm, vias 1 -> 0
- net /BOODOO_BOARD1/SDA: track 56.3 -> 0.00 mm
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- removed copper zone on B.Cu, net GND
- removed copper zone on F.Cu, net GND
Other:
- board outline removed
- board text removed: "Master of Muppets presents Dr. Teeth and the Electic Mayhem Rev 1"

Commit message: Bigger and noisier
Migrates code form Arduino IDE into Platform.io IDE.
Refactor code to accommodate AD5993R. The plan is to test with it and if feasible use AD5992R which is the SPI version of it.
Adding external dependencies into `lib` folder and not managing them via IDE.
Parts:
- added C1: 0.1uf, Capacitor_THT:C_Disc_D5.0mm_W2.5mm_P5.00mm, F.Cu at (-101.8, 62.8)
- added C2: 0.1uf, Capacitor_THT:C_Disc_D5.0mm_W2.5mm_P5.00mm, F.Cu at (-101.8, 66.8)
- added C3: 0.1uf, Capacitor_THT:C_Disc_D5.0mm_W2.5mm_P5.00mm, F.Cu at (-101.8, 70.9)
- added C4: 1uf, Capacitor_THT:C_Disc_D5.0mm_W2.5mm_P5.00mm, F.Cu at (-101.8, 74.9)
- added C5: 0.1uf, Capacitor_THT:C_Disc_D5.0mm_W2.5mm_P5.00mm, F.Cu at (-101.8, 79.0)
- added DAC0: MCP4728, Package_SO:MSOP-10_3x3mm_P0.5mm, F.Cu at (21.8, 40.6)
- added DAC1: MCP4728, Package_SO:MSOP-10_3x3mm_P0.5mm, F.Cu at (86.4, 40.1)
- added DAC2: MCP4728, Package_SO:MSOP-10_3x3mm_P0.5mm, F.Cu at (175.3, 44.2)
- added Eurorack1: ~, Connector_IDC:IDC-Header_2x08_P2.54mm_Vertical, F.Cu at (-110.1, 66.9)
- added OUT_CV1: ACJM-MV35-2S, PCM_4ms_Jack:ACJM-MV35-2S_Mono_Vert_Switch, F.Cu at (135.9, 17.3)
- added OUT_CV10: ACJM-MV35-2S, PCM_4ms_Jack:ACJM-MV35-2S_Mono_Vert_Switch, F.Cu at (209.1, 17.8)
- added OUT_CV11: ACJM-MV35-2S, PCM_4ms_Jack:ACJM-MV35-2S_Mono_Vert_Switch, F.Cu at (257.6, 21.3)
- added OUT_CV12: ACJM-MV35-2S, PCM_4ms_Jack:ACJM-MV35-2S_Mono_Vert_Switch, F.Cu at (282.4, 20.3)
- added OUT_CV2: ACJM-MV35-2S, PCM_4ms_Jack:ACJM-MV35-2S_Mono_Vert_Switch, F.Cu at (117.1, 17.3)
- added OUT_CV3: ACJM-MV35-2S, PCM_4ms_Jack:ACJM-MV35-2S_Mono_Vert_Switch, F.Cu at (178.3, 17.8)
- added OUT_CV4: ACJM-MV35-2S, PCM_4ms_Jack:ACJM-MV35-2S_Mono_Vert_Switch, F.Cu at (156.5, 19.3)
- added OUT_CV5: ACJM-MV35-2S, PCM_4ms_Jack:ACJM-MV35-2S_Mono_Vert_Switch, F.Cu at (47.8, 16.3)
- added OUT_CV6: ACJM-MV35-2S, PCM_4ms_Jack:ACJM-MV35-2S_Mono_Vert_Switch, F.Cu at (68.1, 16.8)
- added OUT_CV7: ACJM-MV35-2S, PCM_4ms_Jack:ACJM-MV35-2S_Mono_Vert_Switch, F.Cu at (26.4, 17.3)
- added OUT_CV8: ACJM-MV35-2S, PCM_4ms_Jack:ACJM-MV35-2S_Mono_Vert_Switch, F.Cu at (86.9, 17.8)
- added OUT_CV9: ACJM-MV35-2S, PCM_4ms_Jack:ACJM-MV35-2S_Mono_Vert_Switch, F.Cu at (233.2, 20.3)
- added OpAmp0: TL074, Package_DIP:DIP-14_W7.62mm_Socket, F.Cu at (47.2, 44.2)
- added OpAmp1: TL074, Package_DIP:DIP-14_W7.62mm_Socket, F.Cu at (114.3, 44.2)
- added OpAmp2: TL074, Package_DIP:DIP-14_W7.62mm_Socket, F.Cu at (204.0, 40.6)
- added R1: 1k, Resistor_THT:R_Axial_DIN0204_L3.6mm_D1.6mm_P1.90mm_Vertical, F.Cu at (103.8, 38.6)
- added R10: 47k, Resistor_THT:R_Axial_DIN0204_L3.6mm_D1.6mm_P1.90mm_Vertical, F.Cu at (130.5, 54.0)
- added R11: 1k, Resistor_THT:R_Axial_DIN0204_L3.6mm_D1.6mm_P1.90mm_Vertical, F.Cu at (106.2, 67.1)
- added R12: 1k, Resistor_THT:R_Axial_DIN0204_L3.6mm_D1.6mm_P1.90mm_Vertical, F.Cu at (131.7, 68.6)
- added R13: 10k, Resistor_THT:R_Axial_DIN0204_L3.6mm_D1.6mm_P1.90mm_Vertical, F.Cu at (-3.42, 64.0)
- added R14: 100k, Resistor_THT:R_Axial_DIN0204_L3.6mm_D1.6mm_P1.90mm_Vertical, F.Cu at (-9.01, 51.8)
- added R15: 10k, Resistor_THT:R_Axial_DIN0204_L3.6mm_D1.6mm_P1.90mm_Vertical, F.Cu at (-15.6, 38.1)
- added R16: 100k, Resistor_THT:R_Axial_DIN0204_L3.6mm_D1.6mm_P1.90mm_Vertical, F.Cu at (74.3, 37.6)
- added R17: 10k, Resistor_THT:R_Axial_DIN0204_L3.6mm_D1.6mm_P1.90mm_Vertical, F.Cu at (82.9, 48.8)
- added R18: 100k, Resistor_THT:R_Axial_DIN0204_L3.6mm_D1.6mm_P1.90mm_Vertical, F.Cu at (165.2, 52.3)
- added R19: 10k, Resistor_THT:R_Axial_DIN0204_L3.6mm_D1.6mm_P1.90mm_Vertical, F.Cu at (80.9, 34.0)
- added R2: 1k, Resistor_THT:R_Axial_DIN0204_L3.6mm_D1.6mm_P1.90mm_Vertical, F.Cu at (124.6, 39.1)
- added R20: 10k, Resistor_THT:R_Axial_DIN0204_L3.6mm_D1.6mm_P1.90mm_Vertical, F.Cu at (166.2, 46.7)
- added R21: 10k, Resistor_THT:R_Axial_DIN0204_L3.6mm_D1.6mm_P1.90mm_Vertical, F.Cu at (164.7, 41.1)
- added R22: 1k, Resistor_THT:R_Axial_DIN0204_L3.6mm_D1.6mm_P1.90mm_Vertical, F.Cu at (45.2, 35.1)
- added R23: 1k, Resistor_THT:R_Axial_DIN0204_L3.6mm_D1.6mm_P1.90mm_Vertical, F.Cu at (59.6, 39.1)
- added R24: 1k, Resistor_THT:R_Axial_DIN0204_L3.6mm_D1.6mm_P1.90mm_Vertical, F.Cu at (195.2, 35.1)
- added R25: 1k, Resistor_THT:R_Axial_DIN0204_L3.6mm_D1.6mm_P1.90mm_Vertical, F.Cu at (213.5, 34.0)
- added R26: 47k, Resistor_THT:R_Axial_DIN0204_L3.6mm_D1.6mm_P1.90mm_Vertical, F.Cu at (40.8, 40.6)
- added R27: 47k, Resistor_THT:R_Axial_DIN0204_L3.6mm_D1.6mm_P1.90mm_Vertical, F.Cu at (60.5, 44.2)
- added R28: 47k, Resistor_THT:R_Axial_DIN0204_L3.6mm_D1.6mm_P1.90mm_Vertical, F.Cu at (185.6, 49.8)
- added R29: 47k, Resistor_THT:R_Axial_DIN0204_L3.6mm_D1.6mm_P1.90mm_Vertical, F.Cu at (219.2, 42.1)
- added R3: 47k, Resistor_THT:R_Axial_DIN0204_L3.6mm_D1.6mm_P1.90mm_Vertical, F.Cu at (105.3, 50.8)
- added R30: 47k, Resistor_THT:R_Axial_DIN0204_L3.6mm_D1.6mm_P1.90mm_Vertical, F.Cu at (24.5, 49.3)
- added R31: 47k, Resistor_THT:R_Axial_DIN0204_L3.6mm_D1.6mm_P1.90mm_Vertical, F.Cu at (59.6, 49.3)
- added R32: 47k, Resistor_THT:R_Axial_DIN0204_L3.6mm_D1.6mm_P1.90mm_Vertical, F.Cu at (192.2, 43.2)
- added R33: 47k, Resistor_THT:R_Axial_DIN0204_L3.6mm_D1.6mm_P1.90mm_Vertical, F.Cu at (231.3, 45.2)
- added R34: 47k, Resistor_THT:R_Axial_DIN0204_L3.6mm_D1.6mm_P1.90mm_Vertical, F.Cu at (23.5, 65.5)
- added R35: 47k, Resistor_THT:R_Axial_DIN0204_L3.6mm_D1.6mm_P1.90mm_Vertical, F.Cu at (73.2, 57.9)
- added R36: 47k, Resistor_THT:R_Axial_DIN0204_L3.6mm_D1.6mm_P1.90mm_Vertical, F.Cu at (191.1, 55.9)
- added R37: 47k, Resistor_THT:R_Axial_DIN0204_L3.6mm_D1.6mm_P1.90mm_Vertical, F.Cu at (219.2, 54.7)
- added R38: 47k, Resistor_THT:R_Axial_DIN0204_L3.6mm_D1.6mm_P1.90mm_Vertical, F.Cu at (37.7, 57.4)
- added R39: 47k, Resistor_THT:R_Axial_DIN0204_L3.6mm_D1.6mm_P1.90mm_Vertical, F.Cu at (61.5, 54.9)
- added R4: 47k, Resistor_THT:R_Axial_DIN0204_L3.6mm_D1.6mm_P1.90mm_Vertical, F.Cu at (120.5, 34.5)
- added R40: 47k, Resistor_THT:R_Axial_DIN0204_L3.6mm_D1.6mm_P1.90mm_Vertical, F.Cu at (181.5, 62.5)
- added R41: 47k, Resistor_THT:R_Axial_DIN0204_L3.6mm_D1.6mm_P1.90mm_Vertical, F.Cu at (233.3, 56.9)
- added R42: 1k, Resistor_THT:R_Axial_DIN0204_L3.6mm_D1.6mm_P1.90mm_Vertical, F.Cu at (51.4, 67.6)
- added R43: 1k, Resistor_THT:R_Axial_DIN0204_L3.6mm_D1.6mm_P1.90mm_Vertical, F.Cu at (66.2, 68.6)
- added R44: 1k, Resistor_THT:R_Axial_DIN0204_L3.6mm_D1.6mm_P1.90mm_Vertical, F.Cu at (192.2, 64.0)
- added R45: 1k, Resistor_THT:R_Axial_DIN0204_L3.6mm_D1.6mm_P1.90mm_Vertical, F.Cu at (220.1, 62.0)
- added R5: 47k, Resistor_THT:R_Axial_DIN0204_L3.6mm_D1.6mm_P1.90mm_Vertical, F.Cu at (98.2, 44.2)
- added R6: 47k, Resistor_THT:R_Axial_DIN0204_L3.6mm_D1.6mm_P1.90mm_Vertical, F.Cu at (126.5, 43.2)
- added R7: 47k, Resistor_THT:R_Axial_DIN0204_L3.6mm_D1.6mm_P1.90mm_Vertical, F.Cu at (97.5, 54.4)
- added R8: 47k, Resistor_THT:R_Axial_DIN0204_L3.6mm_D1.6mm_P1.90mm_Vertical, F.Cu at (144.9, 52.3)
- added R9: 47k, Resistor_THT:R_Axial_DIN0204_L3.6mm_D1.6mm_P1.90mm_Vertical, F.Cu at (102.6, 58.4)
- added T1: Teensy4.1, teensy.pretty-master:Teensy41, F.Cu at (95.8, 107.2)
- added V_REG1: LD1117V50, PCM_4ms_Package_TO:TO-220-3_Vertical, F.Cu at (-89.4, 64.2)

Commit message: Preps for PCB Layout
- PCB Reset;
- Footprint assignment - opting for SMD over THT. I got tired of this much soldering;
- Fixing path for teensy.kicad_sym
- Changed symbols of the 3.5mm jack connector to the usual one seen in Eurorack (thanks for the symbols, 4ms!) ;
Parts:
- removed C1, C2, C3, C5: 0.1uf, Capacitor_THT:C_Disc_D5.0mm_W2.5mm_P5.00mm
- removed C4: 1uf, Capacitor_THT:C_Disc_D5.0mm_W2.5mm_P5.00mm
- removed DAC0, DAC1, DAC2: MCP4728, Package_SO:MSOP-10_3x3mm_P0.5mm
- removed Eurorack1: ~, Connector_IDC:IDC-Header_2x08_P2.54mm_Vertical
- removed OUT_CV1, OUT_CV10, OUT_CV11, OUT_CV12, OUT_CV2, OUT_CV3, OUT_CV4, OUT_CV5, OUT_CV6, OUT_CV7, OUT_CV8, OUT_CV9: ACJM-MV35-2S, PCM_4ms_Jack:ACJM-MV35-2S_Mono_Vert_Switch
- removed OpAmp0, OpAmp1, OpAmp2: TL074, Package_DIP:DIP-14_W7.62mm_Socket
- removed R1, R11, R12, R2, R22, R23, R24, R25, R42, R43, R44, R45: 1k, Resistor_THT:R_Axial_DIN0204_L3.6mm_D1.6mm_P1.90mm_Vertical
- removed R10, R26, R27, R28, R29, R3, R30, R31, R32, R33, R34, R35, R36, R37, R38, R39, R4, R40, R41, R5, R6, R7, R8, R9: 47k, Resistor_THT:R_Axial_DIN0204_L3.6mm_D1.6mm_P1.90mm_Vertical
- removed R13, R15, R17, R19, R20, R21: 10k, Resistor_THT:R_Axial_DIN0204_L3.6mm_D1.6mm_P1.90mm_Vertical
- removed R14, R16, R18: 100k, Resistor_THT:R_Axial_DIN0204_L3.6mm_D1.6mm_P1.90mm_Vertical
- removed T1: Teensy4.1, teensy.pretty-master:Teensy41
- removed V_REG1: LD1117V50, PCM_4ms_Package_TO:TO-220-3_Vertical

Commit message: PCB Preps
Re-assigned footprints;
Placed all symbols in the middle;
Removed instruction to ignore the PCB in the README.manahmanah;
Added a generic placement recommendation file from Sir. Claude;
Ready to start the design;
Parts:
- added C1: 100nF ceramic, PCM_4ms_Capacitor:C_0603, F.Cu at (185.7, 103.7)
- added C10: 100pF_0603_50V, PCM_4ms_Capacitor:C_0603, F.Cu at (165.1, 83.4)
- added C11: 100pF_0603_50V, PCM_4ms_Capacitor:C_0603, F.Cu at (165.1, 86.0)
- added C12: 100pF_0603_50V, PCM_4ms_Capacitor:C_0603, F.Cu at (165.1, 88.7)
- added C13: 100pF_0603_50V, PCM_4ms_Capacitor:C_0603, F.Cu at (141.6, 80.7)
- added C14: 100pF_0603_50V, PCM_4ms_Capacitor:C_0603, F.Cu at (141.6, 83.4)
- added C15: 100pF_0603_50V, PCM_4ms_Capacitor:C_0603, F.Cu at (141.6, 86.0)
- added C16: 100pF_0603_50V, PCM_4ms_Capacitor:C_0603, F.Cu at (141.6, 88.7)
- added C17: 100pF_0603_50V, PCM_4ms_Capacitor:C_0603, F.Cu at (141.6, 103.7)
- added C18: 100pF_0603_50V, PCM_4ms_Capacitor:C_0603, F.Cu at (141.6, 106.3)
- added C19: 100pF_0603_50V, PCM_4ms_Capacitor:C_0603, F.Cu at (141.6, 109.0)
- added C2: 10µF ceramic, PCM_4ms_Capacitor:C_0805, F.Cu at (187.3, 112.6)
- added C20: 100pF_0603_50V, PCM_4ms_Capacitor:C_0603, F.Cu at (141.6, 111.6)
- added C21: 100nF_0603_16V, PCM_4ms_Capacitor:C_0603, F.Cu at (181.8, 88.2)
- added C22: 10uF_0805_25V, PCM_4ms_Capacitor:C_0805, F.Cu at (181.8, 91.0)
- added C23: 100nF_0603_16V, PCM_4ms_Capacitor:C_0603, F.Cu at (134.8, 126.7)
- added C24: 10uF_0805_25V, PCM_4ms_Capacitor:C_0805, F.Cu at (134.8, 129.4)
- added C25: 100nF_0603_16V, PCM_4ms_Capacitor:C_0603, F.Cu at (183.0, 126.7)
- added C26: 10uF_0805_25V, PCM_4ms_Capacitor:C_0805, F.Cu at (182.9, 129.4)
- added C27: 100nF_0603_16V, PCM_4ms_Capacitor:C_0603, F.Cu at (128.6, 134.2)
- added C28: 10uF_0805_25V, PCM_4ms_Capacitor:C_0805, F.Cu at (128.5, 136.9)
- added C29: 100nF_0603_16V, PCM_4ms_Capacitor:C_0603, F.Cu at (158.3, 136.2)
- added C3: 100nF ceramic, PCM_4ms_Capacitor:C_0603, F.Cu at (185.7, 106.3)
- added C30: 10uF_0805_25V, PCM_4ms_Capacitor:C_0805, F.Cu at (158.2, 138.9)
- added C31: 100nF_0603_16V, PCM_4ms_Capacitor:C_0603, F.Cu at (141.1, 126.7)
- added C32: 10uF_0805_25V, PCM_4ms_Capacitor:C_0805, F.Cu at (141.0, 129.4)
- added C33: 100nF_0603_16V, PCM_4ms_Capacitor:C_0603, F.Cu at (181.8, 80.7)
- added C34: 10uF_0805_25V, PCM_4ms_Capacitor:C_0805, F.Cu at (181.8, 83.5)
- added C35: 100nF_0603_16V, PCM_4ms_Capacitor:C_0603, F.Cu at (128.6, 126.7)
- added C36: 10uF_0805_25V, PCM_4ms_Capacitor:C_0805, F.Cu at (128.5, 129.4)
- added C37: 100nF_0603_16V, PCM_4ms_Capacitor:C_0603, F.Cu at (175.6, 95.7)
- added C38: 10uF_0805_25V, PCM_4ms_Capacitor:C_0805, F.Cu at (175.5, 98.5)
- added C39: 100nF_0603_16V, PCM_4ms_Capacitor:C_0603, F.Cu at (173.8, 136.2)
- added C4: 22uF_0603_16V, PCM_4ms_Capacitor:C_0805, F.Cu at (187.3, 115.5)
- added C40: 10uF_0805_25V, PCM_4ms_Capacitor:C_0805, F.Cu at (173.7, 138.9)
- added C41: 100nF_0603_16V, PCM_4ms_Capacitor:C_0603, F.Cu at (152.1, 136.2)
- added C42: 10uF_0805_25V, PCM_4ms_Capacitor:C_0805, F.Cu at (152.0, 138.9)
- added C43: 100nF_0603_16V, PCM_4ms_Capacitor:C_0603, F.Cu at (181.8, 95.7)
- added C44: 10uF_0805_25V, PCM_4ms_Capacitor:C_0805, F.Cu at (181.8, 98.5)
- added C45: 100nF_0603_16V, PCM_4ms_Capacitor:C_0603, F.Cu at (175.6, 88.2)
- added C46: 10uF_0805_25V, PCM_4ms_Capacitor:C_0805, F.Cu at (175.5, 91.0)
- added C47: 100nF_0603_16V, PCM_4ms_Capacitor:C_0603, F.Cu at (167.5, 136.2)
- added C48: 10uF_0805_25V, PCM_4ms_Capacitor:C_0805, F.Cu at (167.5, 138.9)
- added C49: 100nF_0603_16V, PCM_4ms_Capacitor:C_0603, F.Cu at (183.0, 134.2)
- added C5: 100pF_0603_50V, PCM_4ms_Capacitor:C_0603, F.Cu at (165.1, 103.7)
- added C50: 10uF_0805_25V, PCM_4ms_Capacitor:C_0805, F.Cu at (182.9, 136.9)
- added C51: 100nF_0603_16V, PCM_4ms_Capacitor:C_0603, F.Cu at (175.6, 80.7)
- added C52: 10uF_0805_25V, PCM_4ms_Capacitor:C_0805, F.Cu at (175.5, 83.5)
- added C6: 100pF_0603_50V, PCM_4ms_Capacitor:C_0603, F.Cu at (165.1, 106.3)
- added C7: 100pF_0603_50V, PCM_4ms_Capacitor:C_0603, F.Cu at (165.1, 109.0)
- added C8: 100pF_0603_50V, PCM_4ms_Capacitor:C_0603, F.Cu at (165.1, 111.6)
- added C9: 100pF_0603_50V, PCM_4ms_Capacitor:C_0603, F.Cu at (165.1, 80.7)
- added DAC1: AD5593R, Package_SO:TSSOP-16_4.4x5mm_P0.65mm, F.Cu at (174.5, 128.6)
- added DAC2: AD5593R, Package_SO:TSSOP-16_4.4x5mm_P0.65mm, F.Cu at (159.0, 128.6)
- added J1: Screw_Terminal_01x03, TerminalBlock:TerminalBlock_Xinya_XY308-2.54-3P_1x03_P2.54mm_Horizontal, F.Cu at (176.0, 106.5)
- added J10: 3.5mm_Mono_Switched_SymSmall_0.05, PCM_4ms_Jack:EighthInch_PJ398SM, F.Cu at (117.0, 63.7)
- added J11: 3.5mm_Mono_Switched_SymSmall_0.05, PCM_4ms_Jack:EighthInch_PJ398SM, F.Cu at (117.0, 74.2)
- added J12: 3.5mm_Mono_Switched_SymSmall_0.05, PCM_4ms_Jack:EighthInch_PJ398SM, F.Cu at (117.0, 84.6)
- added J13: 3.5mm_Mono_Switched_SymSmall_0.05, PCM_4ms_Jack:EighthInch_PJ398SM, F.Cu at (117.0, 95.1)
- added J14: 3.5mm_Mono_Switched_SymSmall_0.05, PCM_4ms_Jack:EighthInch_PJ398SM, F.Cu at (117.0, 105.5)
- added J15: 3.5mm_Mono_Switched_SymSmall_0.05, PCM_4ms_Jack:EighthInch_PJ398SM, F.Cu at (117.0, 116.0)
- added J16: 3.5mm_Mono_Switched_SymSmall_0.05, PCM_4ms_Jack:EighthInch_PJ398SM, F.Cu at (117.0, 126.4)
- added J17: 3.5mm_Mono_Switched_SymSmall_0.05, PCM_4ms_Jack:EighthInch_PJ398SM, F.Cu at (117.0, 136.9)
- added J2: 3.5mm_Mono_Switched_SymSmall_0.05, PCM_4ms_Jack:EighthInch_PJ398SM, F.Cu at (100.5, 63.7)
- added J3: 3.5mm_Mono_Switched_SymSmall_0.05, PCM_4ms_Jack:EighthInch_PJ398SM, F.Cu at (100.5, 74.2)
- added J4: 3.5mm_Mono_Switched_SymSmall_0.05, PCM_4ms_Jack:EighthInch_PJ398SM, F.Cu at (100.5, 84.6)
- added J5: 3.5mm_Mono_Switched_SymSmall_0.05, PCM_4ms_Jack:EighthInch_PJ398SM, F.Cu at (100.5, 95.1)
- added J6: 3.5mm_Mono_Switched_SymSmall_0.05, PCM_4ms_Jack:EighthInch_PJ398SM, F.Cu at (100.5, 105.5)
- added J7: 3.5mm_Mono_Switched_SymSmall_0.05, PCM_4ms_Jack:EighthInch_PJ398SM, F.Cu at (100.5, 116.0)
- added J8: 3.5mm_Mono_Switched_SymSmall_0.05, PCM_4ms_Jack:EighthInch_PJ398SM, F.Cu at (100.5, 126.4)
- added J9: 3.5mm_Mono_Switched_SymSmall_0.05, PCM_4ms_Jack:EighthInch_PJ398SM, F.Cu at (100.5, 136.9)
- added OpAmp1: TL074, Package_SO:SOIC-14_3.9x8.7mm_P1.27mm, F.Cu at (167.2, 118.2)
- added OpAmp2: TL074, Package_SO:SOIC-14_3.9x8.7mm_P1.27mm, F.Cu at (167.2, 95.3)
- added OpAmp3: TL074, Package_SO:SOIC-14_3.9x8.7mm_P1.27mm, F.Cu at (143.7, 95.3)
- added OpAmp4: TL074, Package_SO:SOIC-14_3.9x8.7mm_P1.27mm, F.Cu at (143.7, 118.2)
- added R1: 10k, Resistor_SMD:R_0603_1608Metric_Pad0.98x0.95mm_HandSolder, F.Cu at (167.6, 126.6)
- added R10: 220Ω, Resistor_SMD:R_0603_1608Metric_Pad0.98x0.95mm_HandSolder, F.Cu at (156.4, 103.6)
- added R11: 220Ω, Resistor_SMD:R_0603_1608Metric_Pad0.98x0.95mm_HandSolder, F.Cu at (156.4, 106.1)
- added R12: 1k, Resistor_SMD:R_0603_1608Metric_Pad0.98x0.95mm_HandSolder, F.Cu at (156.4, 108.6)
- added R13: 1k, Resistor_SMD:R_0603_1608Metric_Pad0.98x0.95mm_HandSolder, F.Cu at (156.4, 111.2)
- added R14: 47k, Resistor_SMD:R_0603_1608Metric_Pad0.98x0.95mm_HandSolder, F.Cu at (156.4, 113.7)
- added R15: 47k, Resistor_SMD:R_0603_1608Metric_Pad0.98x0.95mm_HandSolder, F.Cu at (156.4, 116.2)
- added R16: 47k, Resistor_SMD:R_0603_1608Metric_Pad0.98x0.95mm_HandSolder, F.Cu at (160.8, 103.6)
- added R17: 47k, Resistor_SMD:R_0603_1608Metric_Pad0.98x0.95mm_HandSolder, F.Cu at (160.8, 106.1)
- added R18: 220Ω, Resistor_SMD:R_0603_1608Metric_Pad0.98x0.95mm_HandSolder, F.Cu at (160.8, 108.6)
- added R19: 220Ω, Resistor_SMD:R_0603_1608Metric_Pad0.98x0.95mm_HandSolder, F.Cu at (160.8, 111.2)
- added R2: 4.7k, Resistor_SMD:R_0603_1608Metric_Pad0.98x0.95mm_HandSolder, F.Cu at (167.6, 129.1)
- added R20: 1k, Resistor_SMD:R_0603_1608Metric_Pad0.98x0.95mm_HandSolder, F.Cu at (152.1, 80.7)
- added R21: 1k, Resistor_SMD:R_0603_1608Metric_Pad0.98x0.95mm_HandSolder, F.Cu at (152.1, 83.2)
- added R22: 47k, Resistor_SMD:R_0603_1608Metric_Pad0.98x0.95mm_HandSolder, F.Cu at (152.1, 85.7)
- added R23: 47k, Resistor_SMD:R_0603_1608Metric_Pad0.98x0.95mm_HandSolder, F.Cu at (152.1, 88.2)
- added R24: 47k, Resistor_SMD:R_0603_1608Metric_Pad0.98x0.95mm_HandSolder, F.Cu at (152.1, 90.7)
- added R25: 47k, Resistor_SMD:R_0603_1608Metric_Pad0.98x0.95mm_HandSolder, F.Cu at (152.1, 93.2)
- added R26: 220Ω, Resistor_SMD:R_0603_1608Metric_Pad0.98x0.95mm_HandSolder, F.Cu at (156.4, 80.7)
- added R27: 220Ω, Resistor_SMD:R_0603_1608Metric_Pad0.98x0.95mm_HandSolder, F.Cu at (156.4, 83.2)
- added R28: 1k, Resistor_SMD:R_0603_1608Metric_Pad0.98x0.95mm_HandSolder, F.Cu at (156.4, 85.7)
- added R29: 1k, Resistor_SMD:R_0603_1608Metric_Pad0.98x0.95mm_HandSolder, F.Cu at (156.4, 88.2)
- added R3: 4.7k, Resistor_SMD:R_0603_1608Metric_Pad0.98x0.95mm_HandSolder, F.Cu at (167.6, 131.6)
- added R30: 47k, Resistor_SMD:R_0603_1608Metric_Pad0.98x0.95mm_HandSolder, F.Cu at (156.4, 90.7)
- added R31: 47k, Resistor_SMD:R_0603_1608Metric_Pad0.98x0.95mm_HandSolder, F.Cu at (156.4, 93.2)
- added R32: 47k, Resistor_SMD:R_0603_1608Metric_Pad0.98x0.95mm_HandSolder, F.Cu at (160.8, 80.7)
- added R33: 47k, Resistor_SMD:R_0603_1608Metric_Pad0.98x0.95mm_HandSolder, F.Cu at (160.8, 83.2)
- added R34: 220Ω, Resistor_SMD:R_0603_1608Metric_Pad0.98x0.95mm_HandSolder, F.Cu at (160.8, 85.7)
- added R35: 220Ω, Resistor_SMD:R_0603_1608Metric_Pad0.98x0.95mm_HandSolder, F.Cu at (160.8, 88.2)
- added R36: 10k, Resistor_SMD:R_0603_1608Metric_Pad0.98x0.95mm_HandSolder, F.Cu at (152.1, 126.6)
- added R37: 4.7k, Resistor_SMD:R_0603_1608Metric_Pad0.98x0.95mm_HandSolder, F.Cu at (152.1, 129.1)
- added R38: 4.7k, Resistor_SMD:R_0603_1608Metric_Pad0.98x0.95mm_HandSolder, F.Cu at (152.1, 131.6)
- added R39: 1k, Resistor_SMD:R_0603_1608Metric_Pad0.98x0.95mm_HandSolder, F.Cu at (128.6, 80.7)
- added R4: 1k, Resistor_SMD:R_0603_1608Metric_Pad0.98x0.95mm_HandSolder, F.Cu at (152.1, 103.6)
- added R40: 1k, Resistor_SMD:R_0603_1608Metric_Pad0.98x0.95mm_HandSolder, F.Cu at (128.6, 83.2)
- added R41: 47k, Resistor_SMD:R_0603_1608Metric_Pad0.98x0.95mm_HandSolder, F.Cu at (128.6, 85.7)
- added R42: 47k, Resistor_SMD:R_0603_1608Metric_Pad0.98x0.95mm_HandSolder, F.Cu at (128.6, 88.2)
- added R43: 47k, Resistor_SMD:R_0603_1608Metric_Pad0.98x0.95mm_HandSolder, F.Cu at (128.6, 90.7)
- added R44: 47k, Resistor_SMD:R_0603_1608Metric_Pad0.98x0.95mm_HandSolder, F.Cu at (128.6, 93.2)
- added R45: 220Ω, Resistor_SMD:R_0603_1608Metric_Pad0.98x0.95mm_HandSolder, F.Cu at (132.9, 80.7)
- added R46: 220Ω, Resistor_SMD:R_0603_1608Metric_Pad0.98x0.95mm_HandSolder, F.Cu at (132.9, 83.2)
- added R47: 1k, Resistor_SMD:R_0603_1608Metric_Pad0.98x0.95mm_HandSolder, F.Cu at (132.9, 85.7)
- added R48: 1k, Resistor_SMD:R_0603_1608Metric_Pad0.98x0.95mm_HandSolder, F.Cu at (132.9, 88.2)
- added R49: 47k, Resistor_SMD:R_0603_1608Metric_Pad0.98x0.95mm_HandSolder, F.Cu at (132.9, 90.7)
- added R5: 1k, Resistor_SMD:R_0603_1608Metric_Pad0.98x0.95mm_HandSolder, F.Cu at (152.1, 106.1)
- added R50: 47k, Resistor_SMD:R_0603_1608Metric_Pad0.98x0.95mm_HandSolder, F.Cu at (132.9, 93.2)
- added R51: 47k, Resistor_SMD:R_0603_1608Metric_Pad0.98x0.95mm_HandSolder, F.Cu at (137.3, 80.7)
- added R52: 47k, Resistor_SMD:R_0603_1608Metric_Pad0.98x0.95mm_HandSolder, F.Cu at (137.3, 83.2)
- added R53: 220Ω, Resistor_SMD:R_0603_1608Metric_Pad0.98x0.95mm_HandSolder, F.Cu at (137.3, 85.7)
- added R54: 220Ω, Resistor_SMD:R_0603_1608Metric_Pad0.98x0.95mm_HandSolder, F.Cu at (137.3, 88.2)
- added R55: 1k, Resistor_SMD:R_0603_1608Metric_Pad0.98x0.95mm_HandSolder, F.Cu at (128.6, 103.6)
- added R56: 1k, Resistor_SMD:R_0603_1608Metric_Pad0.98x0.95mm_HandSolder, F.Cu at (128.6, 106.1)
- added R57: 47k, Resistor_SMD:R_0603_1608Metric_Pad0.98x0.95mm_HandSolder, F.Cu at (128.6, 108.6)
- added R58: 47k, Resistor_SMD:R_0603_1608Metric_Pad0.98x0.95mm_HandSolder, F.Cu at (128.6, 111.2)
- added R59: 47k, Resistor_SMD:R_0603_1608Metric_Pad0.98x0.95mm_HandSolder, F.Cu at (128.6, 113.7)
- added R6: 47k, Resistor_SMD:R_0603_1608Metric_Pad0.98x0.95mm_HandSolder, F.Cu at (152.1, 108.6)
- added R60: 47k, Resistor_SMD:R_0603_1608Metric_Pad0.98x0.95mm_HandSolder, F.Cu at (128.6, 116.2)
- added R61: 220Ω, Resistor_SMD:R_0603_1608Metric_Pad0.98x0.95mm_HandSolder, F.Cu at (132.9, 103.6)
- added R62: 220Ω, Resistor_SMD:R_0603_1608Metric_Pad0.98x0.95mm_HandSolder, F.Cu at (132.9, 106.1)
- added R63: 1k, Resistor_SMD:R_0603_1608Metric_Pad0.98x0.95mm_HandSolder, F.Cu at (132.9, 108.6)
- added R64: 1k, Resistor_SMD:R_0603_1608Metric_Pad0.98x0.95mm_HandSolder, F.Cu at (132.9, 111.2)
- added R65: 47k, Resistor_SMD:R_0603_1608Metric_Pad0.98x0.95mm_HandSolder, F.Cu at (132.9, 113.7)
- added R66: 47k, Resistor_SMD:R_0603_1608Metric_Pad0.98x0.95mm_HandSolder, F.Cu at (132.9, 116.2)
- added R67: 47k, Resistor_SMD:R_0603_1608Metric_Pad0.98x0.95mm_HandSolder, F.Cu at (137.3, 103.6)
- added R68: 47k, Resistor_SMD:R_0603_1608Metric_Pad0.98x0.95mm_HandSolder, F.Cu at (137.3, 106.1)
- added R69: 220Ω, Resistor_SMD:R_0603_1608Metric_Pad0.98x0.95mm_HandSolder, F.Cu at (137.3, 108.6)
- added R7: 47k, Resistor_SMD:R_0603_1608Metric_Pad0.98x0.95mm_HandSolder, F.Cu at (152.1, 111.2)
- added R70: 220Ω, Resistor_SMD:R_0603_1608Metric_Pad0.98x0.95mm_HandSolder, F.Cu at (137.3, 111.2)
- added R8: 47k, Resistor_SMD:R_0603_1608Metric_Pad0.98x0.95mm_HandSolder, F.Cu at (152.1, 113.7)
- added R9: 47k, Resistor_SMD:R_0603_1608Metric_Pad0.98x0.95mm_HandSolder, F.Cu at (152.1, 116.2)
- added T1: Teensy4.1, Teensy:Teensy41, F.Cu at (158.8, 67.9)
- added V_REG1: LD1117V50, PCM_4ms_Package_TO:TO-220-3_Vertical, F.Cu at (179.3, 114.6)
