File: hardware/master_of_muppets/teensy_module.kicad_sch (KiCad schematic)
At the start: 1 part, among them T1 Teensy4.1

Commit message: Circuit analysis graphs
It made me realize that i broke the kicad project files that, now are fixed.
Other:
- title: MasterOfMuppets -> master_of_muppets
Changed lines of the file:
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@@
 	(paper "A4")
 	(title_block
-		(title "MasterOfMuppets")
+		(title "master_of_muppets")
 		(rev "0.0.0")
 		(company "y3i12")
@@
 		)
 		(instances
-			(project "MasterOfMuppets"
+			(project "master_of_muppets"
 				(path "/01709e3c-d295-4eba-a9f6-77b38e73bd4a/9146edb4-d9ec-4eb9-99ec-c7182bcc31c9"
 					(reference "#PWR09")
@@
 		)
 		(instances
-			(project "MasterOfMuppets"
+			(project "master_of_muppets"
 				(path "/01709e3c-d295-4eba-a9f6-77b38e73bd4a/9146edb4-d9ec-4eb9-99ec-c7182bcc31c9"
 					(reference "T1")
@@
 		)
 		(instances
-			(project "MasterOfMuppets"
+			(project "master_of_muppets"
 				(path "/01709e3c-d295-4eba-a9f6-77b38e73bd4a/9146edb4-d9ec-4eb9-99ec-c7182bcc31c9"
 					(reference "#PWR010")
@@
 		)
 		(instances
-			(project "MasterOfMuppets"
+			(project "master_of_muppets"
 				(path "/01709e3c-d295-4eba-a9f6-77b38e73bd4a/9146edb4-d9ec-4eb9-99ec-c7182bcc31c9"
 					(reference "#PWR07")
@@
 		)
 		(instances
-			(project "MasterOfMuppets"
+			(project "master_of_muppets"
 				(path "/01709e3c-d295-4eba-a9f6-77b38e73bd4a/9146edb4-d9ec-4eb9-99ec-c7182bcc31c9"
 					(reference "#PWR08")
