File: hardware/master_of_muppets/unripple_module.kicad_sch (KiCad schematic)
At the start: 2 parts

Commit message: Circuit analysis graphs
It made me realize that i broke the kicad project files that, now are fixed.
Other:
- title: MasterOfMuppets -> master_of_muppets
Changed lines of the file:
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@@
 	(paper "A5")
 	(title_block
-		(title "MasterOfMuppets")
+		(title "master_of_muppets")
 		(rev "0.0.0")
 		(company "y3i12")
@@
 		)
 		(instances
-			(project "MasterOfMuppets"
+			(project "master_of_muppets"
 				(path "/01709e3c-d295-4eba-a9f6-77b38e73bd4a/2605ff3f-ff92-4fa9-a945-25b3be4a890c/1ebaab9f-3adf-4ab6-b6c9-964263e520cd"
 					(reference "C26")
@@
 		)
 		(instances
-			(project "MasterOfMuppets"
+			(project "master_of_muppets"
 				(path "/01709e3c-d295-4eba-a9f6-77b38e73bd4a/2605ff3f-ff92-4fa9-a945-25b3be4a890c/1ebaab9f-3adf-4ab6-b6c9-964263e520cd"
 					(reference "#PWR057")
@@
 		)
 		(instances
-			(project "MasterOfMuppets"
+			(project "master_of_muppets"
 				(path "/01709e3c-d295-4eba-a9f6-77b38e73bd4a/2605ff3f-ff92-4fa9-a945-25b3be4a890c/1ebaab9f-3adf-4ab6-b6c9-964263e520cd"
 					(reference "C25")
