File: hardware/master_of_muppets/master_of_muppets.kicad_pcb (KiCad board)
At the start: 2 copper layers, 147 parts, among them J1 Screw_Terminal_01x03, J10 3.5mm_Mono_Switched_SymSmall_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, J11 3.5mm_Mono_Switched_SymSmall_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, J12 3.5mm_Mono_Switched_SymSmall_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, J13 3.5mm_Mono_Switched_SymSmall_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, J14 3.5mm_Mono_Switched_SymSmall_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, J15 3.5mm_Mono_Switched_SymSmall_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, J16 3.5mm_Mono_Switched_SymSmall_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, J17 3.5mm_Mono_Switched_SymSmall_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, J2 3.5mm_Mono_Switched_SymSmall_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

Commit message: unripple, amp and dac modules routed
Other:
- copper layers 2 -> 4
Changed lines of the file:
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@@
 	(layers
 		(0 "F.Cu" signal)
+		(4 "In1.Cu" signal)
+		(6 "In2.Cu" signal)
 		(2 "B.Cu" signal)
 		(9 "F.Adhes" user "F.Adhesive")
@@
 			)
 			(layer "dielectric 1"
-				(type "core")
+				(type "prepreg")
 				(color "FR4 natural")
-				(thickness 1.459)
+				(thickness 0.1)
 				(material "FR4")
 				(epsilon_r 4.5)
+				(loss_tangent 0.02)
+			)
+			(layer "In1.Cu"
+				(type "copper")
+				(thickness 0.035)
+			)
+			(layer "dielectric 2"
+				(type "core")
+				(thickness 1.189)
+				(material "FR4")
+				(epsilon_r 4.5)
+				(loss_tangent 0.02)
+			)
+			(layer "In2.Cu"
+				(type "copper")
+				(thickness 0.035)
+			)
+			(layer "dielectric 3"
+				(type "prepreg")
+				(thickness 0.1)
+				(material "FR4")
+				(epsilon_r 4.5)
