File: hardware/master_of_muppets/master_of_muppets.kicad_sch (KiCad schematic)
At the start: 6 parts, among them J1 Screw_Terminal_01x03

Commit message: Circuit analysis graphs
It made me realize that i broke the kicad project files that, now are fixed.
Other:
- title: MasterOfMuppets -> master_of_muppets
Changed lines of the file:
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@@
 	(paper "A5")
 	(title_block
-		(title "MasterOfMuppets")
+		(title "master_of_muppets")
 		(date "localtime();")
 		(rev "0.0.0")
@@
 		)
 		(instances
-			(project "MasterOfMuppets"
+			(project "master_of_muppets"
 				(path "/01709e3c-d295-4eba-a9f6-77b38e73bd4a"
 					(reference "J1")
@@
 		)
 		(instances
-			(project "MasterOfMuppets"
+			(project "master_of_muppets"
 				(path "/01709e3c-d295-4eba-a9f6-77b38e73bd4a"
 					(reference "#PWR06")
@@
 		)
 		(instances
-			(project "MasterOfMuppets"
+			(project "master_of_muppets"
 				(path "/01709e3c-d295-4eba-a9f6-77b38e73bd4a"
 					(reference "#PWR01")
@@
 		)
 		(instances
-			(project "MasterOfMuppets"
+			(project "master_of_muppets"
 				(path "/01709e3c-d295-4eba-a9f6-77b38e73bd4a"
 					(reference "#PWR02")
@@
 		)
 		(instances
-			(project "MasterOfMuppets"
+			(project "master_of_muppets"
 				(path "/01709e3c-d295-4eba-a9f6-77b38e73bd4a"
 					(reference "#PWR03")
@@
 		)
 		(instances
-			(project "MasterOfMuppets"
+			(project "master_of_muppets"
 				(path "/01709e3c-d295-4eba-a9f6-77b38e73bd4a"
 					(reference "#PWR04")
@@
 		)
 		(instances
-			(project "MasterOfMuppets"
+			(project "master_of_muppets"
 				(path "/01709e3c-d295-4eba-a9f6-77b38e73bd4a"
 					(reference "C1")
@@
 		)
 		(instances
-			(project "MasterOfMuppets"
+			(project "master_of_muppets"
 				(path "/01709e3c-d295-4eba-a9f6-77b38e73bd4a"
 					(reference "V_REG1")
@@
 		)
 		(instances
-			(project "MasterOfMuppets"
+			(project "master_of_muppets"
 				(path "/01709e3c-d295-4eba-a9f6-77b38e73bd4a"
 					(reference "C3")
@@
 		)
 		(instances
-			(project "MasterOfMuppets"
+			(project "master_of_muppets"
 				(path "/01709e3c-d295-4eba-a9f6-77b38e73bd4a"
 					(reference "C2")
@@
 		)
 		(instances
-			(project "MasterOfMuppets"
+			(project "master_of_muppets"
 				(path "/01709e3c-d295-4eba-a9f6-77b38e73bd4a"
 					(reference "#PWR05")
@@
 		)
 		(instances
-			(project "MasterOfMuppets"
+			(project "master_of_muppets"
 				(path "/01709e3c-d295-4eba-a9f6-77b38e73bd4a"
 					(reference "C4")
@@
 		)
 		(instances
-			(project "MasterOfMuppets"
+			(project "master_of_muppets"
 				(path "/01709e3c-d295-4eba-a9f6-77b38e73bd4a"
 					(page "5")
@@
 		)
 		(instances
-			(project "MasterOfMuppets"
+			(project "master_of_muppets"
 				(path "/01709e3c-d295-4eba-a9f6-77b38e73bd4a"
 					(page "2")
@@
 		)
 		(instances
-			(project "MasterOfMuppets"
+			(project "master_of_muppets"
 				(path "/01709e3c-d295-4eba-a9f6-77b38e73bd4a"
 					(page "1")
@@
 		)
 		(instances
-			(project "MasterOfMuppets"
+			(project "master_of_muppets"
 				(path "/01709e3c-d295-4eba-a9f6-77b38e73bd4a"
 					(page "23")
@@
 		)
 		(instances
-			(project "MasterOfMuppets"
+			(project "master_of_muppets"
 				(path "/01709e3c-d295-4eba-a9f6-77b38e73bd4a"
 					(page "25")

Commit message: Making the boards truly hierarchical using projectinstances plugin
https://github.com/OfficialDyray/projectinstances
Other:
- sheet DAC_MODULE: file dac_module.kicad_sch -> dac_module/dac_module.kicad_sch
- sheet DAC_MODULE1: file dac_module.kicad_sch -> dac_module/dac_module.kicad_sch
- sheet JACK_SHEET: file jack_sheet.kicad_sch -> jack_sheet/jack_sheet.kicad_sch
- sheet JACK_SHEET1: file jack_sheet.kicad_sch -> jack_sheet/jack_sheet.kicad_sch
- sheet TEENSY_MODULE: file teensy_module.kicad_sch -> teensy_module/teensy_module.kicad_sch
Changed lines of the file:
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@@
 			)
 		)
-		(property "Sheetfile" "dac_module.kicad_sch"
+		(property "Sheetfile" "dac_module/dac_module.kicad_sch"
 			(at 60.325 109.1696 0)
 			(effects
@@
 			)
 		)
-		(property "Sheetfile" "dac_module.kicad_sch"
+		(property "Sheetfile" "dac_module/dac_module.kicad_sch"
 			(at 20.32 108.5346 0)
 			(effects
@@
 			)
 		)
-		(property "Sheetfile" "teensy_module.kicad_sch"
+		(property "Sheetfile" "teensy_module/teensy_module.kicad_sch"
 			(at 62.1796 40.64 90)
 			(effects
@@
 			)
 		)
-		(property "Sheetfile" "jack_sheet.kicad_sch"
+		(property "Sheetfile" "jack_sheet/jack_sheet.kicad_sch"
 			(at 73.025 109.1696 0)
 			(effects
@@
 			)
 		)
-		(property "Sheetfile" "jack_sheet.kicad_sch"
+		(property "Sheetfile" "jack_sheet/jack_sheet.kicad_sch"
 			(at 33.02 108.5346 0)
 			(effects

Commit message: pcb work
Parts:
- removed C1, C3: 100nF ceramic, PCM_4ms_Capacitor:C_0603, symbol Device:C
- removed C2: 10µF ceramic, PCM_4ms_Capacitor:C_0805, symbol Device:C
- removed C4: 22uF_0603_16V, PCM_4ms_Capacitor:C_0805, symbol PCM_4ms_Capacitor:22uF_0603_16V
- removed J1: Screw_Terminal_01x03, TerminalBlock:TerminalBlock_Xinya_XY308-2.54-3P_1x03_P2.54mm_Horizontal, symbol Connector:Screw_Terminal_01x03
- removed V_REG1: LD1117V50, PCM_4ms_Package_TO:TO-220-3_Vertical, symbol Regulator_Linear:LD1117S50TR_SOT223
Other:
- added sheet POWER_MODULE (power_module/power_module.kicad_sch)
- added sheet SCREW_TERMINAL (power_in_screw_header_module/power_in_screw_header_module.kicad_sch)
