File: hardware/master_of_muppets/amp_module/amp_module.kicad_pcb (KiCad board)
At the start: 2 copper layers, 25 parts, among them U1 TL074CNS

Commit message: unripple, amp and dac modules routed
Parts:
- moved RO_U1B1 1.31 mm to (94.2, 67.0), turned to 0 degrees
- moved RO_U1A1 1.20 mm to (94.2, 53.5), turned to 0 degrees
- moved RO_U1C1 1.18 mm to (99.5, 67.0), turned to 180 degrees
- moved RO_U1D1 1.11 mm to (99.5, 53.5), turned to 180 degrees
Other:
- copper layers 2 -> 4
