File: hardware/master_of_muppets/dac_module/dac_module.kicad_pcb (KiCad board)
At the start: 4 copper layers, 62 parts, among them U1 TL074CNS, U2 TL074CNS

Commit message: pcb work
Parts:
- added J+12V1: PinHeader_1x04_P1.00mm_Vertical, Connector_PinHeader_1.00mm:PinHeader_1x04_P1.00mm_Vertical, F.Cu at (49.0, 27.0)
- added J-12V1: PinHeader_1x04_P1.00mm_Vertical, Connector_PinHeader_1.00mm:PinHeader_1x04_P1.00mm_Vertical, F.Cu at (40.0, 55.8)
- added J-12V2: PinHeader_1x04_P1.00mm_Vertical, Connector_PinHeader_1.00mm:PinHeader_1x04_P1.00mm_Vertical, F.Cu at (64.2, 55.8)
- added JO_1234: PinHeader_1x04_P1.00mm_Vertical, Connector_PinHeader_1.00mm:PinHeader_1x04_P1.00mm_Vertical, F.Cu at (25.5, 39.5)
- added JO_5678: PinHeader_1x04_P1.00mm_Vertical, Connector_PinHeader_1.00mm:PinHeader_1x04_P1.00mm_Vertical, F.Cu at (75.8, 39.8)
- added J_GCD1: PinHeader_1x03_P1.00mm_Vertical, Connector_PinHeader_1.00mm:PinHeader_1x03_P1.00mm_Vertical, F.Cu at (44.8, 42.8)
- added J_VCR1: PinHeader_1x03_P1.00mm_Vertical, Connector_PinHeader_1.00mm:PinHeader_1x03_P1.00mm_Vertical, F.Cu at (55.5, 42.8)
- moved C14 41.2 mm to (36.1, 51.4)
- moved CI_U1A2 41.2 mm to (40.2, 31.4)
- moved CI_U1B2 41.2 mm to (30.1, 31.4)
- moved CI_U1C1 41.2 mm to (60.8, 51.1)
- moved CI_U1D1 41.2 mm to (70.9, 51.1)
- moved RD_U1A1 41.2 mm to (70.9, 33.4)
- moved RD_U1A2 41.2 mm to (40.2, 33.3)
- moved RD_U1B1 41.2 mm to (60.8, 33.4)
- moved RD_U1B2 41.2 mm to (30.0, 33.3)
- moved RD_U1C1 41.2 mm to (60.8, 49.2)
- moved RD_U1C2 41.2 mm to (30.0, 49.2)
- moved RD_U1D1 41.2 mm to (70.9, 49.2)
- moved RD_U1D2 41.2 mm to (40.2, 49.2)
- moved RF_U1A1 41.2 mm to (70.9, 35.3)
- moved RF_U1B1 41.2 mm to (60.8, 35.3)
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Routing:
- net +12V: track 36.4 -> 70.1 mm
- net -12V: track 37.2 -> 70.3 mm
- net /~{RESET}: track 8.85 -> 7.28 mm, vias 1 -> 0
- net /SDA: track 3.98 -> 2.41 mm, vias 1 -> 0
- net GND: track 63.1 -> 63.8 mm, vias 29 -> 28
- net /AMP2_DAC1/INPUT_3: track 18.3 -> 19.0 mm
- net /~{CHIP_SELECT}: track 13.3 -> 12.6 mm, vias 1 -> 0
- net /SCL: track 7.72 -> 7.05 mm, vias 1 -> 0
- net /AMP2_DAC1/INPUT_1: track 21.4 -> 22.0 mm
- net /AMP2_DAC1/INPUT_4: track 22.3 -> 22.9 mm
- net VCC: vias 1 -> 0
