File: hardware/master_of_muppets/dac_module/dac_module.kicad_sch (KiCad schematic)
At the start: 4 parts

Commit message: Making the boards truly hierarchical using projectinstances plugin
https://github.com/OfficialDyray/projectinstances
Other:
- sheet AMP_MODULE: file amp_module.kicad_sch -> ../amp_module/amp_module.kicad_sch
- sheet AMP_MODULE1: file amp_module.kicad_sch -> ../amp_module/amp_module.kicad_sch
- sheet UNRIPPLE_MODULE: file unripple_module.kicad_sch -> ../unripple_module/unripple_module.kicad_sch
- sheet UNRIPPLE_MODULE1: file unripple_module.kicad_sch -> ../unripple_module/unripple_module.kicad_sch
- sheet UNRIPPLE_MODULE2: file unripple_module.kicad_sch -> ../unripple_module/unripple_module.kicad_sch
- sheet UNRIPPLE_MODULE3: file unripple_module.kicad_sch -> ../unripple_module/unripple_module.kicad_sch
Changed lines of the file:
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@@
 			)
 		)
-		(property "Sheetfile" "amp_module.kicad_sch"
+		(property "Sheetfile" "../amp_module/amp_module.kicad_sch"
 			(at 109.22 75.5146 0)
 			(effects
@@
 			)
 		)
-		(property "Sheetfile" "unripple_module.kicad_sch"
+		(property "Sheetfile" "../unripple_module/unripple_module.kicad_sch"
 			(at 69.85 76.1496 0)
 			(effects
@@
 			)
 		)
-		(property "Sheetfile" "amp_module.kicad_sch"
+		(property "Sheetfile" "../amp_module/amp_module.kicad_sch"
 			(at 109.22 85.6746 0)
 			(effects
@@
 			)
 		)
-		(property "Sheetfile" "unripple_module.kicad_sch"
+		(property "Sheetfile" "../unripple_module/unripple_module.kicad_sch"
 			(at 69.85 83.7696 0)
 			(effects
@@
 			)
 		)
-		(property "Sheetfile" "unripple_module.kicad_sch"
+		(property "Sheetfile" "../unripple_module/unripple_module.kicad_sch"
 			(at 101.6 60.9096 0)
 			(effects
@@
 			)
 		)
-		(property "Sheetfile" "unripple_module.kicad_sch"
+		(property "Sheetfile" "../unripple_module/unripple_module.kicad_sch"
 			(at 69.85 88.8496 0)
 			(effects

Commit message: unripple, amp and dac modules routed
Parts:
- renumbered R2 to RCP_DAC1, R3 to RDP_DAC1, R1 to RRP_DAC1
Other:
- sheet AMP_MODULE renamed AMP1_DAC1
- sheet AMP_MODULE1 renamed AMP2_DAC1
Changed lines of the file:
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@@
+				)
+			)
+			(project "dac_module"
+				(path "/177cfd6a-1ed3-4511-a0a7-a5da522e26c3"
+					(reference "DAC1")
+					(unit 1)
 				)
 			)
@@
 		(on_board yes)
 		(dnp no)
-		(property "Reference" "#PWR011"
+		(property "Reference" "#PWR01"
 			(at 93.98 41.91 0)
 			(effects
@@
 				(path "/01709e3c-d295-4eba-a9f6-77b38e73bd4a/60709206-8158-4f80-9acc-4f76df38190b"
 					(reference "#PWR011")
+					(unit 1)
+				)
+			)
+			(project "dac_module"
+				(path "/177cfd6a-1ed3-4511-a0a7-a5da522e26c3"
+					(reference "#PWR01")
 					(unit 1)
 				)
@@
 		(dnp no)
 		(fields_autoplaced yes)
-		(property "Reference" "R3"
+		(property "Reference" "RDP_DAC1"
 			(at 83.82 31.7499 0)
 			(effects
@@
 				(path "/01709e3c-d295-4eba-a9f6-77b38e73bd4a/60709206-8158-4f80-9acc-4f76df38190b"
 					(reference "R3")
+					(unit 1)
+				)
+			)
+			(project "dac_module"
+				(path "/177cfd6a-1ed3-4511-a0a7-a5da522e26c3"
+					(reference "RDP_DAC1")
 					(unit 1)
 				)
@@
 		(dnp no)
 		(fields_autoplaced yes)
-		(property "Reference" "#PWR012"
+		(property "Reference" "#PWR02"
 			(at 96.52 97.79 0)
 			(effects
@@
 				(path "/01709e3c-d295-4eba-a9f6-77b38e73bd4a/60709206-8158-4f80-9acc-4f76df38190b"
 					(reference "#PWR012")
+					(unit 1)
+				)
+			)
+			(project "dac_module"
+				(path "/177cfd6a-1ed3-4511-a0a7-a5da522e26c3"
+					(reference "#PWR02")
 					(unit 1)
 				)
@@
 		(dnp no)
 		(fields_autoplaced yes)
-		(property "Reference" "R1"
+		(property "Reference" "RRP_DAC1"
 			(at 66.04 31.7499 0)
 			(effects
@@
 				(path "/01709e3c-d295-4eba-a9f6-77b38e73bd4a/60709206-8158-4f80-9acc-4f76df38190b"
 					(reference "R1")
+					(unit 1)
+				)
+			)
+			(project "dac_module"
+				(path "/177cfd6a-1ed3-4511-a0a7-a5da522e26c3"
+					(reference "RRP_DAC1")
 					(unit 1)
 				)
@@
 		(dnp no)
 		(fields_autoplaced yes)
-		(property "Reference" "R2"
+		(property "Reference" "RCP_DAC1"
 			(at 74.93 31.7499 0)
 			(effects
@@
 				(path "/01709e3c-d295-4eba-a9f6-77b38e73bd4a/60709206-8158-4f80-9acc-4f76df38190b"
 					(reference "R2")
+					(unit 1)
+				)
+			)
+			(project "dac_module"
+				(path "/177cfd6a-1ed3-4511-a0a7-a5da522e26c3"
+					(reference "RCP_DAC1")
 					(unit 1)
 				)
@@
 			(color 0 0 0 0.0000)
 		)
-		(property "Sheetname" "AMP_MODULE"
+		(property "Sheetname" "AMP1_DAC1"
 			(at 117.475 64.008 0)
 			(effects
@@
 				)
 				(path "/01709e3c-d295-4eba-a9f6-77b38e73bd4a/2605ff3f-ff92-4fa9-a945-25b3be4a890c"
+					(page "6")
+				)
+			)
+			(project "dac_module"
+				(path "/177cfd6a-1ed3-4511-a0a7-a5da522e26c3"
 					(page "6")
 				)
@@
 				)
 			)
+			(project "dac_module"
+				(path "/177cfd6a-1ed3-4511-a0a7-a5da522e26c3"
+					(page "2")
+				)
+			)
 		)
 	)
@@
 			(color 0 0 0 0.0000)
 		)
-		(property "Sheetname" "AMP_MODULE1"
+		(property "Sheetname" "AMP2_DAC1"
 			(at 117.348 87.122 0)
 			(effects
@@
 				(path "/01709e3c-d295-4eba-a9f6-77b38e73bd4a/2605ff3f-ff92-4fa9-a945-25b3be4a890c"
 					(page "7")
+				)
+			)
+			(project "dac_module"
+				(path "/177cfd6a-1ed3-4511-a0a7-a5da522e26c3"
+					(page "9")
 				)
 			)
@@
 				)
 			)
+			(project "dac_module"
+				(path "/177cfd6a-1ed3-4511-a0a7-a5da522e26c3"
+					(page "3")
+				)
+			)
 		)
 	)
@@
 				)
 			)
+			(project "dac_module"
+				(path "/177cfd6a-1ed3-4511-a0a7-a5da522e26c3"
+					(page "5")
+				)
+			)
 		)
 	)
@@
 				)
 			)
-		)
-	)
+			(project "dac_module"
+				(path "/177cfd6a-1ed3-4511-a0a7-a5da522e26c3"
+					(page "4")
+				)
+			)
+		)
+	)
+	(sheet_instances
+		(path "/"
+			(page "1")
+		)
+	)
+	(embedded_fonts no)
 )

Commit message: pcb work
Parts:
- added J+12V1, J-12V1, J-12V2, JO_1234, JO_5678: PinHeader_1x04_P1.00mm_Vertical, Connector_PinHeader_1.00mm:PinHeader_1x04_P1.00mm_Vertical, symbol Connector:Conn_01x04_Pin
- added J_GCD1, J_VCR1: PinHeader_1x03_P1.00mm_Vertical, Connector_PinHeader_1.00mm:PinHeader_1x03_P1.00mm_Vertical, symbol Connector:Conn_01x03_Pin
Other:
- sheet AMP1_DAC1 ports: added +12V, -12V, GND; removed none
- sheet AMP2_DAC1 ports: added +12V, -12V, GND; removed none
